File: wyse-mod-pcb/wyse-mod-pcb.kicad_sch (KiCad schematic)
At the start: 4 parts, among them J1 RJ9, J2 Handwire, SW1 Reset Switch, U1 Arduino Pro Micro

Commit message: Finished first revision of the PCB
Parts:
- removed U1: Arduino Pro Micro, Arduino:Sparkfun_Pro_Micro, symbol Arduinos:Sparkfun_Pro_Micro
- added U1: ProMicro, Keebio:ArduinoProMicro, symbol Keebio:ProMicro
Connections:
- net +5V: now also U1.21 (VCC)
- net CLK: now also U1.5 (2/PD1)
- net DATA: now also U1.6 (3/PD0)
- net GND: now also U1.23 (GND), U1.3 (GND), U1.4 (GND)
- net RST: now also U1.22 (RST)
- no-connect marks 0 -> 17
